Commit message: fu line detection, regresa codigo para deteccion de polilineas a version original

File: src/autonomos_description/urdf/autonomos.xacro (robot description, xacro)
@@ -21,6 +21,7 @@
   </material>
   <!-- properties -->
-  <xacro:property name="ancho" value="0.005" />
+  <xacro:property name="ancho" value="0.01" />
   <xacro:property name="radio" value="0.020" />
+  <xacro:property name="mu" value="1" />
   <xacro:macro name="inertial_matrix" params="mass">
       <inertial>
@@ -43,4 +44,15 @@
         <material name="Green"/>
     </visual>
+  </xacro:macro>
+  <xacro:macro name="friccion_rueda" params="mu">
+      <surface>
+        <bounce restitution_coefficient=".2" />
+        <friction>
+          <ode mu="${mu}" mu2="${mu}" fdir1="1 0 0" slip1="0" slip2="0" />
+        </friction>
+        <contact>
+          <ode/>
+        </contact>
+      </surface>
   </xacro:macro>
   <xacro:macro name="transmission_block" params="joint_name">
@@ -149,5 +161,6 @@
     <xacro:visual_rueda length="${ancho}" radius="${radio}"/>
     <xacro:collision_rueda length="${ancho}" radius="${radio}"/>
-    <xacro:inertial_matrix mass="0.001"/>
+    <xacro:inertial_matrix mass="0.01"/>
+    <xacro:friccion_rueda mu="${mu}" />
   </link>
   <joint name="back_left_wheel_joint" type="revolute">
@@ -164,5 +177,6 @@
      <xacro:visual_rueda length="${ancho}" radius="${radio}"/>
      <xacro:collision_rueda length="${ancho}" radius="${radio}"/>
-     <xacro:inertial_matrix mass="0.001"/>
+     <xacro:inertial_matrix mass="0.01"/>
+     <xacro:friccion_rueda mu="${mu}" />
   </link>
   <joint name="back_right_wheel_joint" type="revolute">
@@ -224,5 +238,6 @@
     <xacro:visual_rueda length="${ancho}" radius="${radio}"/>
     <xacro:collision_rueda length="${ancho}" radius="${radio}"/>
-    <xacro:inertial_matrix mass="0.001"/>
+    <xacro:inertial_matrix mass="0.01"/>
+    <xacro:friccion_rueda mu="${mu}" />
   </link>
   <joint name="front_left_wheel_joint" type="revolute">
@@ -261,5 +276,6 @@
     <xacro:visual_rueda length="${ancho}" radius="${radio}"/>
     <xacro:collision_rueda length="${ancho}" radius="${radio}"/>
-    <xacro:inertial_matrix mass="0.001"/>
+    <xacro:inertial_matrix mass="0.01"/>
+    <xacro:friccion_rueda mu="${mu}" />
   </link>
   <joint name="front_right_wheel_joint" type="revolute">
